Commit message: Updated wattson description

File: wattson_description/urdf/phobos_generated.urdf (robot description, URDF)
Before this commit: robot Wattson, 17 links, 16 joints
Links:
- removed link link_head_pitch
- removed link link_head_roll
- removed link link_head_yaw
- removed link link_left_forearm
- removed link link_left_hand
- removed link link_left_shoulder
- removed link link_left_shoulder_x
- removed link link_left_upper_arm
- removed link link_left_wrist
- removed link link_left_wrist_x
- removed link link_right_forearm
- removed link link_right_hand
- removed link link_right_shoulder
- removed link link_right_shoulder_x
- removed link link_right_upper_arm
- removed link link_right_wrist
- added link left_forearm_link; collision cylinder length=0.20945 radius=0.04750; visual mesh filename=package://wattson_description/meshes/stl/left_forearm.stl scale=1.00000 1.00000 1.00000
- added link left_shoulder_link; collision cylinder length=0.15394 radius=0.05750; visual mesh filename=package://wattson_description/meshes/stl/left_shoulder.stl scale=1.00000 1.00000 1.00000
- added link left_shoulder_x_link; collision cylinder length=0.20945 radius=0.04750; visual mesh filename=package://wattson_description/meshes/stl/left_shoulder_x.stl scale=1.00000 1.00000 1.00000
- added link left_upper_arm_link; collision cylinder length=0.17294 radius=0.04749; visual mesh filename=package://wattson_description/meshes/stl/left_upper_arm.stl scale=1.00000 1.00000 1.00000
- added link left_wrist_connection_link; collision cylinder length=0.06115 radius=0.02500; visual mesh filename=package://wattson_description/meshes/stl/left_wrist_connect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 scale=1.00000 1.00000 1.00000
- added link left_wrist_link; collision cylinder length=0.06989 radius=0.03505; visual mesh filename=package://wattson_description/meshes/stl/left_wrist.stl scale=1.00000 1.00000 1.00000
- added link left_wrist_x_link; collision cylinder length=0.04097 radius=0.03682; visual mesh filename=package://wattson_description/meshes/stl/left_hand.stl scale=1.00000 1.00000 1.00000
- added link right_forearm_link; collision cylinder length=0.20945 radius=0.04750; visual mesh filename=package://wattson_description/meshes/stl/right_forearm.stl scale=1.00000 1.00000 1.00000
- added link right_shoulder_link; collision cylinder length=0.15394 radius=0.05750; visual mesh filename=package://wattson_description/meshes/stl/right_shoulder.stl scale=1.00000 1.00000 1.00000
- added link right_shoulder_x_link; collision cylinder length=0.20945 radius=0.04750; visual mesh filename=package://wattson_description/meshes/stl/right_shoulder_x.s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 scale=1.00000 1.00000 1.00000
- added link right_upper_arm_link; collision cylinder length=0.17294 radius=0.04749; visual mesh filename=package://wattson_description/meshes/stl/right_upper_arm.stl scale=1.00000 1.00000 1.00000
- added link right_wrist_connection_link; collision cylinder length=0.06115 radius=0.02500; visual mesh filename=package://wattson_description/meshes/stl/right_wrist_connec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 scale=1.00000 1.00000 1.00000
- added link right_wrist_link; collision cylinder length=0.06989 radius=0.03505; visual mesh filename=package://wattson_description/meshes/stl/right_wrist.stl scale=1.00000 1.00000 1.00000
- added link right_wrist_x_link; collision cylinder length=0.04097 radius=0.03682; visual mesh filename=package://wattson_description/meshes/stl/right_hand.stl scale=1.00000 1.00000 1.00000
- link link_torso: geometry collision box size=0.20600 0.09000 0.08500; visual mesh filename=package://wattson_description/meshes/stl/left_shoulder_conn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 scale=1.00000 1.00000 1.00000
Joints:
- removed joint joint_head_pitch
- removed joint joint_head_roll
- removed joint joint_head_yaw
- added joint joint_right_wrist_pitch: type revolute, parent right_wrist_link, child right_wrist_connection_link, origin xyz=0.00045 0.00005 0.05499 rpy=1.79848 -1.57080 1.34311, axis 0.00000 0.00000 1.00000, limit lower=-3.14000 upper=3.14000 effort=0.00000 velocity=0.00000
- joint joint_left_arm_yaw: child link_left_upper_arm -> left_upper_arm_link; origin xyz=-0.00020 0.12745 0.01486 rpy=1.57080 0.00000 0.00000 -> xyz=-0.00717 0.16307 -0.02474 rpy=1.57080 0.00000 0.00000; parent link_left_shoulder_x -> left_shoulder_x_link
- joint joint_left_elbow_pitch: child link_left_forearm -> left_forearm_link; origin xyz=0.00011 -0.00027 -0.23600 rpy=-0.00000 1.57080 0.00000 -> xyz=-0.02455 0.00813 -0.12544 rpy=0.00000 1.57080 0.00000; parent link_left_upper_arm -> left_upper_arm_link
- joint joint_left_forearm_yaw: child link_left_wrist -> left_wrist_link; origin xyz=0.09363 0.00002 -0.00011 rpy=-0.00000 -1.57080 0.00000 -> xyz=0.16300 -0.00751 0.02462 rpy=0.00000 -1.57080 0.00000; parent link_left_forearm -> left_forearm_link
- joint joint_left_shoulder_pitch: child link_left_shoulder -> left_shoulder_link; origin xyz=-0.16356 0.00077 0.19342 rpy=-3.14159 -1.04720 -0.00000 -> xyz=-0.13450 -0.00005 -0.00000 rpy=-0.00000 1.57080 0.00000
- joint joint_left_shoulder_roll: child link_left_shoulder_x -> left_shoulder_x_link; origin xyz=0.00011 0.00077 -0.10785 rpy=1.57080 -1.04720 0.00000 -> xyz=0.00750 0.02422 -0.10644 rpy=-1.57080 -1.57080 0.00000; parent link_left_shoulder -> left_shoulder_link
- joint joint_left_wrist_pitch: child link_left_wrist_x -> left_wrist_connection_link; origin xyz=0.00110 -0.00019 -0.17400 rpy=-0.00000 1.57080 0.00000 -> xyz=-0.00045 -0.00005 -0.05499 rpy=0.00000 1.57080 0.00000; parent link_left_wrist -> left_wrist_link
- joint joint_left_wrist_roll: child link_left_hand -> left_wrist_x_link; origin xyz=0.00002 0.02290 0.00009 rpy=2.42926 1.57080 -2.28313 -> xyz=0.02994 -0.00000 0.00000 rpy=-1.57080 -1.57080 0.00000; parent link_left_wrist_x -> left_wrist_connection_link
- joint joint_right_arm_yaw: child link_right_upper_arm -> right_upper_arm_link; origin xyz=0.00750 -0.13650 0.00800 rpy=1.57080 0.00000 0.00000 -> xyz=0.00717 -0.16307 0.02474 rpy=1.57080 0.00000 0.00000; parent link_right_shoulder_x -> right_shoulder_x_link
- joint joint_right_elbow_pitch: child link_right_forearm -> right_forearm_link; origin xyz=0.00800 -0.00750 0.13550 rpy=1.79848 -1.57080 1.34311 -> xyz=0.02455 -0.00813 0.12544 rpy=1.79848 -1.57080 1.34311; parent link_right_upper_arm -> right_upper_arm_link
- joint joint_right_forearm_yaw: child link_right_wrist -> right_wrist_link; origin xyz=0.12550 -0.00750 -0.00800 rpy=-3.14159 -1.57080 0.00000 -> xyz=0.16300 -0.00751 -0.02462 rpy=-3.14159 -1.57080 0.00000; parent link_right_forearm -> right_forearm_link
- joint joint_right_shoulder_pitch: child link_right_shoulder -> right_shoulder_link; origin xyz=0.16554 0.00000 0.17223 rpy=-0.00000 1.57080 0.00000 -> xyz=0.13454 -0.00005 -0.00000 rpy=-0.00000 1.57080 0.00000
- joint joint_right_shoulder_roll: child link_right_shoulder_x -> right_shoulder_x_link; origin xyz=0.00750 0.00800 0.09550 rpy=1.57080 -1.57080 0.00000 -> xyz=0.00750 0.02422 0.10644 rpy=1.57080 -1.57080 0.00000; parent link_right_shoulder -> right_shoulder_link
- joint joint_right_wrist_roll: child link_right_hand -> right_wrist_x_link; origin xyz=0.00000 -0.03732 0.15088 rpy=-1.57080 0.00000 3.14159 -> xyz=0.02994 -0.00000 -0.00000 rpy=1.57080 -1.57080 0.00000; parent link_right_wrist -> right_wrist_connection_link

Commit message: Comply with conventions

File: wattson_description/urdf/phobos_generated.urdf (robot description, URDF)
Before this commit: robot Wattson, 15 links, 14 joints
Links:
- removed link left_forearm_link
- removed link left_shoulder_link
- removed link left_shoulder_x_link
- removed link left_upper_arm_link
- removed link left_wrist_connection_link
- removed link left_wrist_link
- removed link left_wrist_x_link
- removed link right_forearm_link
- removed link right_shoulder_link
- removed link right_shoulder_x_link
- removed link right_upper_arm_link
- removed link right_wrist_connection_link
- removed link right_wrist_link
- removed link right_wrist_x_link
- added link link_left_elbow; collision cylinder length=0.20945 radius=0.04750; visual mesh filename=package://wattson_description/meshes/stl/left_forearm.stl scale=1.00000 1.00000 1.00000
- added link link_left_forearm; collision cylinder length=0.06989 radius=0.03505; visual mesh filename=package://wattson_description/meshes/stl/left_wrist.stl scale=1.00000 1.00000 1.00000
- added link link_left_hand; collision cylinder length=0.04097 radius=0.03682; visual mesh filename=package://wattson_description/meshes/stl/left_hand.stl scale=1.00000 1.00000 1.00000
- added link link_left_shoulder; collision cylinder length=0.15394 radius=0.05750; visual mesh filename=package://wattson_description/meshes/stl/left_shoulder.stl scale=1.00000 1.00000 1.00000
- added link link_left_shoulder_x; collision cylinder length=0.20945 radius=0.04750; visual mesh filename=package://wattson_description/meshes/stl/left_shoulder_x.stl scale=1.00000 1.00000 1.00000
- added link link_left_upper_arm; collision cylinder length=0.17294 radius=0.04749; visual mesh filename=package://wattson_description/meshes/stl/left_upper_arm.stl scale=1.00000 1.00000 1.00000
- added link link_left_wrist; collision cylinder length=0.06115 radius=0.02500; visual mesh filename=package://wattson_description/meshes/stl/left_wrist_connect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 scale=1.00000 1.00000 1.00000
- added link link_right_elbow; collision cylinder length=0.20945 radius=0.04750; visual mesh filename=package://wattson_description/meshes/stl/right_forearm.stl scale=1.00000 1.00000 1.00000
- added link link_right_forearm; collision cylinder length=0.06989 radius=0.03505; visual mesh filename=package://wattson_description/meshes/stl/right_wrist.stl scale=1.00000 1.00000 1.00000
- added link link_right_hand; collision cylinder length=0.04097 radius=0.03682; visual mesh filename=package://wattson_description/meshes/stl/right_hand.stl scale=1.00000 1.00000 1.00000
- added link link_right_shoulder; collision cylinder length=0.15394 radius=0.05750; visual mesh filename=package://wattson_description/meshes/stl/right_shoulder.stl scale=1.00000 1.00000 1.00000
- added link link_right_shoulder_x; collision cylinder length=0.20945 radius=0.04750; visual mesh filename=package://wattson_description/meshes/stl/right_shoulder_x.s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 scale=1.00000 1.00000 1.00000
- added link link_right_upper_arm; collision cylinder length=0.17294 radius=0.04749; visual mesh filename=package://wattson_description/meshes/stl/right_upper_arm.stl scale=1.00000 1.00000 1.00000
- added link link_right_wrist; collision cylinder length=0.06115 radius=0.02500; visual mesh filename=package://wattson_description/meshes/stl/right_wrist_connec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 scale=1.00000 1.00000 1.00000
Joints:
- joint joint_left_arm_yaw: child left_upper_arm_link -> link_left_upper_arm; parent left_shoulder_x_link -> link_left_shoulder_x
- joint joint_left_elbow_pitch: child left_forearm_link -> link_left_elbow; parent left_upper_arm_link -> link_left_upper_arm
- joint joint_left_forearm_yaw: child left_wrist_link -> link_left_forearm; parent left_forearm_link -> link_left_elbow
- joint joint_left_shoulder_pitch: child left_shoulder_link -> link_left_shoulder
- joint joint_left_shoulder_roll: child left_shoulder_x_link -> link_left_shoulder_x; parent left_shoulder_link -> link_left_shoulder
- joint joint_left_wrist_pitch: child left_wrist_connection_link -> link_left_wrist; parent left_wrist_link -> link_left_forearm
- joint joint_left_wrist_roll: child left_wrist_x_link -> link_left_hand; parent left_wrist_connection_link -> link_left_wrist
- joint joint_right_arm_yaw: child right_upper_arm_link -> link_right_upper_arm; parent right_shoulder_x_link -> link_right_shoulder_x
- joint joint_right_elbow_pitch: child right_forearm_link -> link_right_elbow; parent right_upper_arm_link -> link_right_upper_arm
- joint joint_right_forearm_yaw: child right_wrist_link -> link_right_forearm; parent right_forearm_link -> link_right_elbow
- joint joint_right_shoulder_pitch: child right_shoulder_link -> link_right_shoulder
- joint joint_right_shoulder_roll: child right_shoulder_x_link -> link_right_shoulder_x; parent right_shoulder_link -> link_right_shoulder
- joint joint_right_wrist_pitch: child right_wrist_connection_link -> link_right_wrist; parent right_wrist_link -> link_right_forearm
- joint joint_right_wrist_roll: child right_wrist_x_link -> link_right_hand; parent right_wrist_connection_link -> link_right_wrist

Commit message: Added limits to URDF

File: wattson_description/urdf/phobos_generated.urdf (robot description, URDF)
Before this commit: robot Wattson, 15 links, 14 joints
Joints:
- joint joint_left_arm_yaw: limit lower=-3.14000 upper=3.14000 effort=0.00000 velocity=0.00000 -> lower=-1.30900 upper=0.26180 effort=0.00000 velocity=0.00000
- joint joint_left_elbow_pitch: limit lower=-3.14000 upper=3.14000 effort=0.00000 velocity=0.00000 -> lower=0.00000 upper=1.57080 effort=0.00000 velocity=0.00000
- joint joint_left_forearm_yaw: limit lower=-3.14000 upper=3.14000 effort=0.00000 velocity=0.00000 -> lower=-1.57080 upper=1.57080 effort=0.00000 velocity=0.00000
- joint joint_left_shoulder_pitch: limit lower=-3.14000 upper=3.14000 effort=0.00000 velocity=0.00000 -> lower=0.00000 upper=1.57080 effort=0.00000 velocity=0.00000
- joint joint_left_shoulder_roll: limit lower=-3.14000 upper=3.14000 effort=0.00000 velocity=0.00000 -> lower=0.00000 upper=1.30900 effort=0.00000 velocity=0.00000
- joint joint_left_wrist_pitch: limit lower=-3.14000 upper=3.14000 effort=0.00000 velocity=0.00000 -> lower=-0.69813 upper=0.69813 effort=0.00000 velocity=0.00000
- joint joint_left_wrist_roll: limit lower=-3.14000 upper=3.14000 effort=0.00000 velocity=0.00000 -> lower=-0.69813 upper=0.69813 effort=0.00000 velocity=0.00000
- joint joint_right_arm_yaw: limit lower=-3.14000 upper=3.14000 effort=0.00000 velocity=0.00000 -> lower=-1.30900 upper=0.26180 effort=0.00000 velocity=0.00000
- joint joint_right_elbow_pitch: limit lower=-3.14000 upper=3.14000 effort=0.00000 velocity=0.00000 -> lower=0.00000 upper=1.57080 effort=0.00000 velocity=0.00000
- joint joint_right_forearm_yaw: limit lower=-3.14000 upper=3.14000 effort=0.00000 velocity=0.00000 -> lower=-1.57080 upper=1.57080 effort=0.00000 velocity=0.00000
- joint joint_right_shoulder_pitch: limit lower=-3.14000 upper=3.14000 effort=0.00000 velocity=0.00000 -> lower=0.00000 upper=1.57080 effort=0.00000 velocity=0.00000
- joint joint_right_shoulder_roll: limit lower=-3.14000 upper=3.14000 effort=0.00000 velocity=0.00000 -> lower=0.00000 upper=1.30900 effort=0.00000 velocity=0.00000
- joint joint_right_wrist_pitch: limit lower=-3.14000 upper=3.14000 effort=0.00000 velocity=0.00000 -> lower=-0.69813 upper=0.69813 effort=0.00000 velocity=0.00000
- joint joint_right_wrist_roll: limit lower=-3.14000 upper=3.14000 effort=0.00000 velocity=0.00000 -> lower=-0.69813 upper=0.69813 effort=0.00000 velocity=0.00000

Commit message: Updated URDF

File: wattson_description/urdf/phobos_generated.urdf (robot description, URDF)
Before this commit: robot Wattson, 15 links, 14 joints
Joints:
- joint joint_left_arm_yaw: limit lower=-1.30900 upper=0.26180 effort=0.00000 velocity=0.00000 -> lower=-1.22173 upper=0.34907 effort=0.00000 velocity=0.00000
- joint joint_left_elbow_pitch: limit lower=0.00000 upper=1.57080 effort=0.00000 velocity=0.00000 -> lower=0.00000 upper=1.48353 effort=0.00000 velocity=0.00000
- joint joint_left_shoulder_pitch: limit lower=0.00000 upper=1.57080 effort=0.00000 velocity=0.00000 -> lower=-0.52360 upper=1.04720 effort=0.00000 velocity=0.00000
- joint joint_left_shoulder_roll: limit lower=0.00000 upper=1.30900 effort=0.00000 velocity=0.00000 -> lower=-0.17453 upper=1.30900 effort=0.00000 velocity=0.00000
- joint joint_left_wrist_pitch: limit lower=-0.69813 upper=0.69813 effort=0.00000 velocity=0.00000 -> lower=-0.52360 upper=0.52360 effort=0.00000 velocity=0.00000
- joint joint_left_wrist_roll: limit lower=-0.69813 upper=0.69813 effort=0.00000 velocity=0.00000 -> lower=-0.52360 upper=0.52360 effort=0.00000 velocity=0.00000
- joint joint_right_arm_yaw: limit lower=-1.30900 upper=0.26180 effort=0.00000 velocity=0.00000 -> lower=-1.22173 upper=0.34907 effort=0.00000 velocity=0.00000
- joint joint_right_elbow_pitch: limit lower=0.00000 upper=1.57080 effort=0.00000 velocity=0.00000 -> lower=0.00000 upper=1.48353 effort=0.00000 velocity=0.00000
- joint joint_right_shoulder_pitch: limit lower=0.00000 upper=1.57080 effort=0.00000 velocity=0.00000 -> lower=-0.52360 upper=1.04720 effort=0.00000 velocity=0.00000
- joint joint_right_shoulder_roll: limit lower=0.00000 upper=1.30900 effort=0.00000 velocity=0.00000 -> lower=-0.17453 upper=1.30900 effort=0.00000 velocity=0.00000
- joint joint_right_wrist_pitch: limit lower=-0.69813 upper=0.69813 effort=0.00000 velocity=0.00000 -> lower=-0.52360 upper=0.52360 effort=0.00000 velocity=0.00000
- joint joint_right_wrist_roll: limit lower=-0.69813 upper=0.69813 effort=0.00000 velocity=0.00000 -> lower=-0.52360 upper=0.52360 effort=0.00000 velocity=0.00000
